Commit message: slam gmapping y robot fixed

File: src/mobile_robot/urdf/mobile_robot.xacro (robot description, xacro)
@@ -25,16 +25,16 @@
       />
     </inertial>
-    <collision name='collision'>
-      <origin xyz="0 0 0" rpy=" 0 0 0"/>
-      <geometry>
-        <box size=".4 .2 .1"/>
-      </geometry>
-    </collision>
-    <visual name='chassis_visual'>
-      <origin xyz="0 0 0" rpy=" 0 0 0"/>
-      <geometry>
-        <box size=".4 .2 .1"/>
-      </geometry>
-    </visual>
+  <collision name='collision'>
+  <origin xyz="0 0 0" rpy=" 0 0 0"/>
+  <geometry>
+    <cylinder length="0.1" radius="0.6"/>
+  </geometry>
+  </collision>
+  <visual name='chassis_visual'>
+    <origin xyz="0 0 0" rpy=" 0 0 0"/>
+    <geometry>
+      <cylinder length="0.1" radius="0.3"/>
+    </geometry>
+  </visual>
     <collision name='back_caster_collision'>
       <origin xyz="-0.15 0 -0.05" rpy=" 0 0 0"/>
