Commit message: robot moving pre adjustments

File: src/mobile_robot/urdf/robotuca.xacro (robot description, xacro)
@@ -26,5 +26,5 @@
     </inertial>
     <collision name='collision'>
-      <origin xyz="0 0 0.12" rpy=" 0 0 0"/>
+      <origin xyz="0 0 0.11" rpy=" 0 0 0"/>
       <geometry>
         <cylinder length=".05" radius="0.3"/>
@@ -32,31 +32,7 @@
     </collision>
     <visual name='chassis_visual'>
-      <origin xyz="0 0 0.12" rpy=" 0 0 0"/>
+      <origin xyz="0 0 0.11" rpy=" 0 0 0"/>
       <geometry>
         <cylinder length=".05" radius="0.3"/>
-      </geometry>
-    </visual>
-    <collision name='back_caster_collision'>
-      <origin xyz="-0.15 0 -0.05" rpy=" 0 0 0"/>
-      <geometry>
-        <sphere radius="0.0499"/>
-      </geometry>
-    </collision>
-    <visual name='back_caster_visual'>
-      <origin xyz="-0.15 0 -0.05" rpy=" 0 0 0"/>
-      <geometry>
-        <sphere radius="0.05"/>
-      </geometry>
-    </visual>
-    <collision name='front_caster_collision'>
-      <origin xyz="0.15 0 -0.05" rpy=" 0 0 0"/>
-      <geometry>
-        <sphere radius="0.0499"/>
-      </geometry>
-    </collision>
-    <visual name='front_caster_visual'>
-      <origin xyz="0.15 0 -0.05" rpy=" 0 0 0"/>
-      <geometry>
-        <sphere radius="0.05"/>
       </geometry>
     </visual>
@@ -65,5 +41,5 @@
     <inertial>
       <mass value="5.0"/>
-      <origin xyz="0 0 0" rpy="0 1.5707 1.5707"/>
+      <origin xyz="0 0 0.08" rpy="0 1.5707 1.5707"/>
       <inertia
           ixx="0.1" ixy="0" ixz="0"
@@ -73,5 +49,5 @@
     </inertial>
     <collision name='right_wheel_collision'>
-      <origin xyz="0 0 0" rpy="0 1.5707 1.5707"/>
+      <origin xyz="0 -0.05 0.08" rpy="0 1.5707 1.5707"/>
       <geometry>
         <cylinder length=".055" radius="0.0825"/>
@@ -79,5 +55,5 @@
     </collision>
     <visual name='right_wheel_visual'>
-      <origin xyz="0 0 0" rpy="0 1.5707 1.5707"/>
+      <origin xyz="0 -0.05 0.08" rpy="0 1.5707 1.5707"/>
       <geometry>
         <cylinder length=".055" radius="0.0825"/>
@@ -96,5 +72,5 @@
     <inertial>
       <mass value="5.0"/>
-      <origin xyz="0 0 0" rpy="0 1.5707 1.5707"/>
+      <origin xyz="0 0 0.08" rpy="0 1.5707 1.5707"/>
       <inertia
           ixx="0.1" ixy="0" ixz="0"
@@ -104,5 +80,5 @@
     </inertial>
     <collision name='left_wheel_collision'>
-      <origin xyz="0 0 0" rpy="0 1.5707 1.5707"/>
+      <origin xyz="0 0.05 0.08" rpy="0 1.5707 1.5707"/>
       <geometry>
         <cylinder length=".055" radius="0.0825"/>
@@ -110,5 +86,5 @@
     </collision>
     <visual name='left_wheel_visual'>
-      <origin xyz="0 0 0" rpy="0 1.5707 1.5707"/>
+      <origin xyz="0 0.05 0.08" rpy="0 1.5707 1.5707"/>
       <geometry>
         <cylinder length=".055" radius="0.0825"/>
@@ -164,5 +140,5 @@
     </inertial>
     <collision name='hokuyo_collision'>
-      <origin xyz="0 0 0" rpy="0 0 0"/>
+      <origin xyz="0 0 0.11" rpy="0 0 0"/>
       <geometry>
         <box size=".1 .1 .1"/>
@@ -170,5 +146,5 @@
     </collision>
     <visual name='hokuyo_visual'>
-      <origin xyz="0 0 0" rpy="0 0 0"/>
+      <origin xyz="0 0 0.11" rpy="0 0 0"/>
       <geometry>
          <box size=".1 .1 .1"/>

Commit message: efective base_local_planner navigation

File: src/mobile_robot/urdf/robotuca.xacro (robot description, xacro)
@@ -1,22 +1,18 @@
 <?xml version='1.0'?>
 <robot name="mobile_robot" xmlns:xacro="http://www.ros.org/wiki/xacro">
-  <link name="robot_footprint"></link>
-  <link name="base_link"></link>
-  <xacro:include filename="$(find mobile_robot)/urdf/mobile_robot.gazebo" />
-  <joint name="robot_base__joint" type="fixed">
-    <origin xyz="0 0 0" rpy="0 0 0" />
-    <parent link="robot_footprint"/>
-    <child link="base_link" />
-  </joint>
-  <joint name="robot_footprint_joint" type="fixed">
-    <origin xyz="0 0 0" rpy="0 0 0" />
-    <parent link="base_link"/>
-    <child link="chassis" />
-  </joint>
-  <link name='chassis'>
+  <material name="blue">
+    <color rgba="0 0 0.8 1"/>
+  </material>
+  <material name="black">
+    <color rgba="0 0 0 1"/>
+  </material>
+  <material name="white">
+    <color rgba="1 1 1 1"/>
+  </material>
+  <link name="base_link">
     <pose>0 0 0.1 0 0 0</pose>
     <inertial>
       <mass value="15.0"/>
-      <origin xyz="0.0 0 0" rpy=" 0 0 0"/>
+      <origin xyz="0.0 0 0.11" rpy=" 0 0 0"/>
       <inertia
           ixx="0.1" ixy="0" ixz="0"
@@ -31,9 +27,10 @@
       </geometry>
     </collision>
-    <visual name='chassis_visual'>
+    <visual name='base_link'>
       <origin xyz="0 0 0.11" rpy=" 0 0 0"/>
       <geometry>
         <cylinder length=".05" radius="0.3"/>
       </geometry>
+      <material name="white"/>
     </visual>
   </link>
@@ -41,5 +38,5 @@
     <inertial>
       <mass value="5.0"/>
-      <origin xyz="0 0 0.08" rpy="0 1.5707 1.5707"/>
+      <origin xyz="0 0 0" rpy="0 1.5707 1.5707"/>
       <inertia
           ixx="0.1" ixy="0" ixz="0"
@@ -49,5 +46,5 @@
     </inertial>
     <collision name='right_wheel_collision'>
-      <origin xyz="0 -0.05 0.08" rpy="0 1.5707 1.5707"/>
+      <origin xyz="0 0 0" rpy="0 1.5707 1.5707"/>
       <geometry>
         <cylinder length=".055" radius="0.0825"/>
@@ -55,14 +52,15 @@
     </collision>
     <visual name='right_wheel_visual'>
-      <origin xyz="0 -0.05 0.08" rpy="0 1.5707 1.5707"/>
+      <origin xyz="0 0 0" rpy="0 1.5707 1.5707"/>
       <geometry>
         <cylinder length=".055" radius="0.0825"/>
       </geometry>
+      <material name="black"/>
     </visual>
   </link>
-  <joint type="continuous" name="right_wheel_hinge">
-    <origin xyz="0 -0.27 0" rpy="0 0 0"/>
+  <joint type="fixed" name="right_wheel_hinge">
+    <origin xyz="0 0.27 0.11" rpy="0 0 0"/>
     <child link="right_wheel"/>
-    <parent link="chassis"/>
+    <parent link="base_link"/>
     <axis xyz="0 1 0" rpy="0 0 0"/>
     <limit effort="10000" velocity="1000"/>
@@ -80,5 +78,5 @@
     </inertial>
     <collision name='left_wheel_collision'>
-      <origin xyz="0 0.05 0.08" rpy="0 1.5707 1.5707"/>
+      <origin xyz="0 0 0" rpy="0 1.5707 1.5707"/>
       <geometry>
         <cylinder length=".055" radius="0.0825"/>
@@ -86,19 +84,20 @@
     </collision>
     <visual name='left_wheel_visual'>
-      <origin xyz="0 0.05 0.08" rpy="0 1.5707 1.5707"/>
+      <origin xyz="0 0 0" rpy="0 1.5707 1.5707"/>
       <geometry>
         <cylinder length=".055" radius="0.0825"/>
       </geometry>
+      <material name="black"/>
     </visual>
   </link>
-  <joint type="continuous" name="left_wheel_hinge">
-    <origin xyz="0 0.27 0" rpy="0 0 0"/>
+  <joint type="fixed" name="left_wheel_hinge">
+    <origin xyz="0 -0.27 0.11" rpy="0 0 0"/>
     <child link="left_wheel"/>
-    <parent link="chassis"/>
+    <parent link="base_link"/>
     <axis xyz="0 1 0" rpy="0 0 0"/>
     <limit effort="10000" velocity="1000"/>
     <dynamics damping="1.0" friction="1.0"/>
   </joint>
-  <link name='camera'>
+  <!-- <link name='camera'>
     <inertial>
       <mass value=".1"/>
@@ -128,5 +127,5 @@
     <parent link="chassis"/>
     <axis xyz="0 1 0" rpy="0 0 0"/>
-  </joint>
+  </joint> -->
   <link name='hokuyo'>
     <inertial>
@@ -140,5 +139,5 @@
     </inertial>
     <collision name='hokuyo_collision'>
-      <origin xyz="0 0 0.11" rpy="0 0 0"/>
+      <origin xyz="0 0 0" rpy="0 0 0"/>
       <geometry>
         <box size=".1 .1 .1"/>
@@ -146,14 +145,15 @@
     </collision>
     <visual name='hokuyo_visual'>
-      <origin xyz="0 0 0.11" rpy="0 0 0"/>
+      <origin xyz="0 0 0" rpy="0 0 0"/>
       <geometry>
          <box size=".1 .1 .1"/>
       </geometry>
+      <material name="blue"/>
     </visual>
   </link>
   <joint name="hokuyo_joint" type="fixed">
-    <origin xyz="0 0 0.08" rpy="0 0 0"/>
+    <origin xyz="0 0 0.20" rpy="0 0 0"/>
     <child link="hokuyo"/>
-    <parent link="chassis"/>
+    <parent link="base_link"/>
     <axis xyz="0 1 0" rpy="0 0 0"/>
   </joint>
@@ -166,15 +166,3 @@
     <axis xyz="0 1 0" rpy="0 0 0"/>
   </joint>
-  <gazebo reference="chassis">
-    <material>Gazebo/Blue</material>
-  </gazebo>
-  <gazebo reference="left_wheel">
-    <material>Gazebo/Green</material>
-  </gazebo>
-  <gazebo reference="right_wheel">
-    <material>Gazebo/Green</material>
-  </gazebo>
-  <gazebo reference="camera">
-    <material>Gazebo/Red</material>
-  </gazebo>
 </robot>
